Commit message: updated urdfs

File: assets/leap_hand/plate_macro.xacro (robot description, xacro)
@@ -2,5 +2,5 @@
 <robot name="plate_macro" xmlns:xacro="http://www.ros.org/wiki/xacro">
 <xacro:macro name="plate" params="parent_link id x y z roll pitch yaw">
-    <link name="${parent_link}_sensor_${id}">
+    <link name="plate_${id}_${parent_link}">
         <visual>
           <origin xyz="${x} ${y} ${z}" rpy="${roll} ${pitch} ${yaw}" />
@@ -20,12 +20,12 @@
         <inertial>
             <origin xyz="0 0 0" rpy="0 0 0"/>
-            <mass value="0.00001" />
-            <inertia ixx="1e-9" ixy="0" ixz="0" iyy="1e-9" iyz="0" izz="1e-9" />
+            <mass value="0.0000000000001" />
+            <inertia ixx="1e-10" ixy="0" ixz="0" iyy="1e-10" iyz="0" izz="1e-10" />
         </inertial>
     </link>
-    <joint name="${parent_link}_sensor_${id}_joint" type="fixed">
+    <joint name="plate_${id}_${parent_link}_joint" type="fixed">
       <origin xyz="0 0 0" rpy="0 0 0" />
       <parent link="${parent_link}" />
-      <child link="${parent_link}_sensor_${id}" />
+      <child link="plate_${id}_${parent_link}" />
     </joint>
 </xacro:macro>

File: assets/leap_hand/robot.urdf (robot description, URDF)
Before this commit: robot onshape, 17 links, 16 joints
Links:
- added link plate_0_fingertip, mass 0.0000000000001; collision cylinder length=0.0001 radius=0.001; visual cylinder length=0.0001 radius=0.001
- added link plate_0_fingertip_2, mass 0.0000000000001; collision cylinder length=0.0001 radius=0.001; visual cylinder length=0.0001 radius=0.001
- added link plate_0_fingertip_3, mass 0.0000000000001; collision cylinder length=0.0001 radius=0.001; visual cylinder length=0.0001 radius=0.001
- added link plate_10_fingertip, mass 0.0000000000001; collision cylinder length=0.0001 radius=0.001; visual cylinder length=0.0001 radius=0.001
- added link plate_10_fingertip_2, mass 0.0000000000001; collision cylinder length=0.0001 radius=0.001; visual cylinder length=0.0001 radius=0.001
- added link plate_10_fingertip_3, mass 0.0000000000001; collision cylinder length=0.0001 radius=0.001; visual cylinder length=0.0001 radius=0.001
- added link plate_11_fingertip, mass 0.0000000000001; collision cylinder length=0.0001 radius=0.001; visual cylinder length=0.0001 radius=0.001
- added link plate_11_fingertip_2, mass 0.0000000000001; collision cylinder length=0.0001 radius=0.001; visual cylinder length=0.0001 radius=0.001
- added link plate_11_fingertip_3, mass 0.0000000000001; collision cylinder length=0.0001 radius=0.001; visual cylinder length=0.0001 radius=0.001
- added link plate_1_fingertip, mass 0.0000000000001; collision cylinder length=0.0001 radius=0.001; visual cylinder length=0.0001 radius=0.001
- added link plate_1_fingertip_2, mass 0.0000000000001; collision cylinder length=0.0001 radius=0.001; visual cylinder length=0.0001 radius=0.001
- added link plate_1_fingertip_3, mass 0.0000000000001; collision cylinder length=0.0001 radius=0.001; visual cylinder length=0.0001 radius=0.001
- added link plate_2_fingertip, mass 0.0000000000001; collision cylinder length=0.0001 radius=0.001; visual cylinder length=0.0001 radius=0.001
- added link plate_2_fingertip_2, mass 0.0000000000001; collision cylinder length=0.0001 radius=0.001; visual cylinder length=0.0001 radius=0.001
- added link plate_2_fingertip_3, mass 0.0000000000001; collision cylinder length=0.0001 radius=0.001; visual cylinder length=0.0001 radius=0.001
- added link plate_3_fingertip, mass 0.0000000000001; collision cylinder length=0.0001 radius=0.001; visual cylinder length=0.0001 radius=0.001
- added link plate_3_fingertip_2, mass 0.0000000000001; collision cylinder length=0.0001 radius=0.001; visual cylinder length=0.0001 radius=0.001
- added link plate_3_fingertip_3, mass 0.0000000000001; collision cylinder length=0.0001 radius=0.001; visual cylinder length=0.0001 radius=0.001
- added link plate_4_fingertip, mass 0.0000000000001; collision cylinder length=0.0001 radius=0.001; visual cylinder length=0.0001 radius=0.001
- added link plate_4_fingertip_2, mass 0.0000000000001; collision cylinder length=0.0001 radius=0.001; visual cylinder length=0.0001 radius=0.001
- added link plate_4_fingertip_3, mass 0.0000000000001; collision cylinder length=0.0001 radius=0.001; visual cylinder length=0.0001 radius=0.001
- added link plate_5_fingertip, mass 0.0000000000001; collision cylinder length=0.0001 radius=0.001; visual cylinder length=0.0001 radius=0.001
- added link plate_5_fingertip_2, mass 0.0000000000001; collision cylinder length=0.0001 radius=0.001; visual cylinder length=0.0001 radius=0.001
- added link plate_5_fingertip_3, mass 0.0000000000001; collision cylinder length=0.0001 radius=0.001; visual cylinder length=0.0001 radius=0.001
- added link plate_6_fingertip, mass 0.0000000000001; collision cylinder length=0.0001 radius=0.001; visual cylinder length=0.0001 radius=0.001
- added link plate_6_fingertip_2, mass 0.0000000000001; collision cylinder length=0.0001 radius=0.001; visual cylinder length=0.0001 radius=0.001
- added link plate_6_fingertip_3, mass 0.0000000000001; collision cylinder length=0.0001 radius=0.001; visual cylinder length=0.0001 radius=0.001
- added link plate_7_fingertip, mass 0.0000000000001; collision cylinder length=0.0001 radius=0.001; visual cylinder length=0.0001 radius=0.001
- added link plate_7_fingertip_2, mass 0.0000000000001; collision cylinder length=0.0001 radius=0.001; visual cylinder length=0.0001 radius=0.001
- added link plate_7_fingertip_3, mass 0.0000000000001; collision cylinder length=0.0001 radius=0.001; visual cylinder length=0.0001 radius=0.001
- added link plate_8_fingertip, mass 0.0000000000001; collision cylinder length=0.0001 radius=0.001; visual cylinder length=0.0001 radius=0.001
- added link plate_8_fingertip_2, mass 0.0000000000001; collision cylinder length=0.0001 radius=0.001; visual cylinder length=0.0001 radius=0.001
- added link plate_8_fingertip_3, mass 0.0000000000001; collision cylinder length=0.0001 radius=0.001; visual cylinder length=0.0001 radius=0.001
- added link plate_9_fingertip, mass 0.0000000000001; collision cylinder length=0.0001 radius=0.001; visual cylinder length=0.0001 radius=0.001
- added link plate_9_fingertip_2, mass 0.0000000000001; collision cylinder length=0.0001 radius=0.001; visual cylinder length=0.0001 radius=0.001
- added link plate_9_fingertip_3, mass 0.0000000000001; collision cylinder length=0.0001 radius=0.001; visual cylinder length=0.0001 radius=0.001
Joints:
- added joint plate_0_fingertip_2_joint: type fixed, parent fingertip_2, child plate_0_fingertip_2, origin xyz=0 0 0 rpy=0 0 0
- added joint plate_0_fingertip_3_joint: type fixed, parent fingertip_3, child plate_0_fingertip_3, origin xyz=0 0 0 rpy=0 0 0
- added joint plate_0_fingertip_joint: type fixed, parent fingertip, child plate_0_fingertip, origin xyz=0 0 0 rpy=0 0 0
- added joint plate_10_fingertip_2_joint: type fixed, parent fingertip_2, child plate_10_fingertip_2, origin xyz=0 0 0 rpy=0 0 0
- added joint plate_10_fingertip_3_joint: type fixed, parent fingertip_3, child plate_10_fingertip_3, origin xyz=0 0 0 rpy=0 0 0
- added joint plate_10_fingertip_joint: type fixed, parent fingertip, child plate_10_fingertip, origin xyz=0 0 0 rpy=0 0 0
- added joint plate_11_fingertip_2_joint: type fixed, parent fingertip_2, child plate_11_fingertip_2, origin xyz=0 0 0 rpy=0 0 0
- added joint plate_11_fingertip_3_joint: type fixed, parent fingertip_3, child plate_11_fingertip_3, origin xyz=0 0 0 rpy=0 0 0
- added joint plate_11_fingertip_joint: type fixed, parent fingertip, child plate_11_fingertip, origin xyz=0 0 0 rpy=0 0 0
- added joint plate_1_fingertip_2_joint: type fixed, parent fingertip_2, child plate_1_fingertip_2, origin xyz=0 0 0 rpy=0 0 0
- added joint plate_1_fingertip_3_joint: type fixed, parent fingertip_3, child plate_1_fingertip_3, origin xyz=0 0 0 rpy=0 0 0
- added joint plate_1_fingertip_joint: type fixed, parent fingertip, child plate_1_fingertip, origin xyz=0 0 0 rpy=0 0 0
- added joint plate_2_fingertip_2_joint: type fixed, parent fingertip_2, child plate_2_fingertip_2, origin xyz=0 0 0 rpy=0 0 0
- added joint plate_2_fingertip_3_joint: type fixed, parent fingertip_3, child plate_2_fingertip_3, origin xyz=0 0 0 rpy=0 0 0
- added joint plate_2_fingertip_joint: type fixed, parent fingertip, child plate_2_fingertip, origin xyz=0 0 0 rpy=0 0 0
- added joint plate_3_fingertip_2_joint: type fixed, parent fingertip_2, child plate_3_fingertip_2, origin xyz=0 0 0 rpy=0 0 0
- added joint plate_3_fingertip_3_joint: type fixed, parent fingertip_3, child plate_3_fingertip_3, origin xyz=0 0 0 rpy=0 0 0
- added joint plate_3_fingertip_joint: type fixed, parent fingertip, child plate_3_fingertip, origin xyz=0 0 0 rpy=0 0 0
- added joint plate_4_fingertip_2_joint: type fixed, parent fingertip_2, child plate_4_fingertip_2, origin xyz=0 0 0 rpy=0 0 0
- added joint plate_4_fingertip_3_joint: type fixed, parent fingertip_3, child plate_4_fingertip_3, origin xyz=0 0 0 rpy=0 0 0
- added joint plate_4_fingertip_joint: type fixed, parent fingertip, child plate_4_fingertip, origin xyz=0 0 0 rpy=0 0 0
- added joint plate_5_fingertip_2_joint: type fixed, parent fingertip_2, child plate_5_fingertip_2, origin xyz=0 0 0 rpy=0 0 0
- added joint plate_5_fingertip_3_joint: type fixed, parent fingertip_3, child plate_5_fingertip_3, origin xyz=0 0 0 rpy=0 0 0
- added joint plate_5_fingertip_joint: type fixed, parent fingertip, child plate_5_fingertip, origin xyz=0 0 0 rpy=0 0 0
- added joint plate_6_fingertip_2_joint: type fixed, parent fingertip_2, child plate_6_fingertip_2, origin xyz=0 0 0 rpy=0 0 0
- added joint plate_6_fingertip_3_joint: type fixed, parent fingertip_3, child plate_6_fingertip_3, origin xyz=0 0 0 rpy=0 0 0
- added joint plate_6_fingertip_joint: type fixed, parent fingertip, child plate_6_fingertip, origin xyz=0 0 0 rpy=0 0 0
- added joint plate_7_fingertip_2_joint: type fixed, parent fingertip_2, child plate_7_fingertip_2, origin xyz=0 0 0 rpy=0 0 0
- added joint plate_7_fingertip_3_joint: type fixed, parent fingertip_3, child plate_7_fingertip_3, origin xyz=0 0 0 rpy=0 0 0
- added joint plate_7_fingertip_joint: type fixed, parent fingertip, child plate_7_fingertip, origin xyz=0 0 0 rpy=0 0 0
- added joint plate_8_fingertip_2_joint: type fixed, parent fingertip_2, child plate_8_fingertip_2, origin xyz=0 0 0 rpy=0 0 0
- added joint plate_8_fingertip_3_joint: type fixed, parent fingertip_3, child plate_8_fingertip_3, origin xyz=0 0 0 rpy=0 0 0
- added joint plate_8_fingertip_joint: type fixed, parent fingertip, child plate_8_fingertip, origin xyz=0 0 0 rpy=0 0 0
- added joint plate_9_fingertip_2_joint: type fixed, parent fingertip_2, child plate_9_fingertip_2, origin xyz=0 0 0 rpy=0 0 0
- added joint plate_9_fingertip_3_joint: type fixed, parent fingertip_3, child plate_9_fingertip_3, origin xyz=0 0 0 rpy=0 0 0
- added joint plate_9_fingertip_joint: type fixed, parent fingertip, child plate_9_fingertip, origin xyz=0 0 0 rpy=0 0 0

File: assets/leap_hand/robot.urdf.xacro (robot description, xacro)
@@ -1,10 +1,4 @@
 <robot name="onshape" xmlns:xacro="http://www.ros.org/wiki/xacro">
 <xacro:include filename="/home/control-lab/LEAP_Hand_Sim/assets/leap_hand/plate_macro.xacro"/>
-<link name="world"/>
-<joint name="palm_joint" type="fixed">
-<origin xyz="0 0 0" rpy="0 3.14 0" />
-<parent link="world" />
-<child link="palm_lower" />
-</joint>
 <link name="palm_lower">
 <visual>
