Commit message: updated urdfs for all sensors

File: assets/leap_hand/robot.urdf (robot description, URDF)
Before this commit: robot onshape, 53 links, 52 joints
Links:
- added link plate_10_palm_lower, mass 0.0000000000001; collision cylinder length=0.0001 radius=0.001; visual cylinder length=0.0001 radius=0.001
- added link plate_11_palm_lower, mass 0.0000000000001; collision cylinder length=0.0001 radius=0.001; visual cylinder length=0.0001 radius=0.001
- added link plate_12_palm_lower, mass 0.0000000000001; collision cylinder length=0.0001 radius=0.001; visual cylinder length=0.0001 radius=0.001
- added link plate_13_palm_lower, mass 0.0000000000001; collision cylinder length=0.0001 radius=0.001; visual cylinder length=0.0001 radius=0.001
- added link plate_14_palm_lower, mass 0.0000000000001; collision cylinder length=0.0001 radius=0.001; visual cylinder length=0.0001 radius=0.001
- added link plate_15_palm_lower, mass 0.0000000000001; collision cylinder length=0.0001 radius=0.001; visual cylinder length=0.0001 radius=0.001
- added link plate_16_palm_lower, mass 0.0000000000001; collision cylinder length=0.0001 radius=0.001; visual cylinder length=0.0001 radius=0.001
- added link plate_17_palm_lower, mass 0.0000000000001; collision cylinder length=0.0001 radius=0.001; visual cylinder length=0.0001 radius=0.001
- added link plate_18_palm_lower, mass 0.0000000000001; collision cylinder length=0.0001 radius=0.001; visual cylinder length=0.0001 radius=0.001
- added link plate_19_palm_lower, mass 0.0000000000001; collision cylinder length=0.0001 radius=0.001; visual cylinder length=0.0001 radius=0.001
- added link plate_1_palm_lower, mass 0.0000000000001; collision cylinder length=0.0001 radius=0.001; visual cylinder length=0.0001 radius=0.001
- added link plate_1_thumb_fingertip, mass 0.0000000000001; collision cylinder length=0.0001 radius=0.001; visual cylinder length=0.0001 radius=0.001
- added link plate_20_palm_lower, mass 0.0000000000001; collision cylinder length=0.0001 radius=0.001; visual cylinder length=0.0001 radius=0.001
- added link plate_21_palm_lower, mass 0.0000000000001; collision cylinder length=0.0001 radius=0.001; visual cylinder length=0.0001 radius=0.001
- added link plate_22_palm_lower, mass 0.0000000000001; collision cylinder length=0.0001 radius=0.001; visual cylinder length=0.0001 radius=0.001
- added link plate_23_palm_lower, mass 0.0000000000001; collision cylinder length=0.0001 radius=0.001; visual cylinder length=0.0001 radius=0.001
- added link plate_24_palm_lower, mass 0.0000000000001; collision cylinder length=0.0001 radius=0.001; visual cylinder length=0.0001 radius=0.001
- added link plate_25_palm_lower, mass 0.0000000000001; collision cylinder length=0.0001 radius=0.001; visual cylinder length=0.0001 radius=0.001
- added link plate_2_palm_lower, mass 0.0000000000001; collision cylinder length=0.0001 radius=0.001; visual cylinder length=0.0001 radius=0.001
- added link plate_2_thumb_fingertip, mass 0.0000000000001; collision cylinder length=0.0001 radius=0.001; visual cylinder length=0.0001 radius=0.001
- added link plate_3_palm_lower, mass 0.0000000000001; collision cylinder length=0.0001 radius=0.001; visual cylinder length=0.0001 radius=0.001
- added link plate_3_thumb_fingertip, mass 0.0000000000001; collision cylinder length=0.0001 radius=0.001; visual cylinder length=0.0001 radius=0.001
- added link plate_4_palm_lower, mass 0.0000000000001; collision cylinder length=0.0001 radius=0.001; visual cylinder length=0.0001 radius=0.001
- added link plate_4_thumb_fingertip, mass 0.0000000000001; collision cylinder length=0.0001 radius=0.001; visual cylinder length=0.0001 radius=0.001
- added link plate_5_palm_lower, mass 0.0000000000001; collision cylinder length=0.0001 radius=0.001; visual cylinder length=0.0001 radius=0.001
- added link plate_5_thumb_fingertip, mass 0.0000000000001; collision cylinder length=0.0001 radius=0.001; visual cylinder length=0.0001 radius=0.001
- added link plate_6_palm_lower, mass 0.0000000000001; collision cylinder length=0.0001 radius=0.001; visual cylinder length=0.0001 radius=0.001
- added link plate_6_thumb_fingertip, mass 0.0000000000001; collision cylinder length=0.0001 radius=0.001; visual cylinder length=0.0001 radius=0.001
- added link plate_7_palm_lower, mass 0.0000000000001; collision cylinder length=0.0001 radius=0.001; visual cylinder length=0.0001 radius=0.001
- added link plate_7_thumb_fingertip, mass 0.0000000000001; collision cylinder length=0.0001 radius=0.001; visual cylinder length=0.0001 radius=0.001
- added link plate_8_palm_lower, mass 0.0000000000001; collision cylinder length=0.0001 radius=0.001; visual cylinder length=0.0001 radius=0.001
- added link plate_8_thumb_fingertip, mass 0.0000000000001; collision cylinder length=0.0001 radius=0.001; visual cylinder length=0.0001 radius=0.001
- added link plate_9_palm_lower, mass 0.0000000000001; collision cylinder length=0.0001 radius=0.001; visual cylinder length=0.0001 radius=0.001
- added link plate_9_thumb_fingertip, mass 0.0000000000001; collision cylinder length=0.0001 radius=0.001; visual cylinder length=0.0001 radius=0.001
Joints:
- added joint plate_10_palm_lower_joint: type fixed, parent palm_lower, child plate_10_palm_lower, origin xyz=0 0 0 rpy=0 0 0
- added joint plate_11_palm_lower_joint: type fixed, parent palm_lower, child plate_11_palm_lower, origin xyz=0 0 0 rpy=0 0 0
- added joint plate_12_palm_lower_joint: type fixed, parent palm_lower, child plate_12_palm_lower, origin xyz=0 0 0 rpy=0 0 0
- added joint plate_13_palm_lower_joint: type fixed, parent palm_lower, child plate_13_palm_lower, origin xyz=0 0 0 rpy=0 0 0
- added joint plate_14_palm_lower_joint: type fixed, parent palm_lower, child plate_14_palm_lower, origin xyz=0 0 0 rpy=0 0 0
- added joint plate_15_palm_lower_joint: type fixed, parent palm_lower, child plate_15_palm_lower, origin xyz=0 0 0 rpy=0 0 0
- added joint plate_16_palm_lower_joint: type fixed, parent palm_lower, child plate_16_palm_lower, origin xyz=0 0 0 rpy=0 0 0
- added joint plate_17_palm_lower_joint: type fixed, parent palm_lower, child plate_17_palm_lower, origin xyz=0 0 0 rpy=0 0 0
- added joint plate_18_palm_lower_joint: type fixed, parent palm_lower, child plate_18_palm_lower, origin xyz=0 0 0 rpy=0 0 0
- added joint plate_19_palm_lower_joint: type fixed, parent palm_lower, child plate_19_palm_lower, origin xyz=0 0 0 rpy=0 0 0
- added joint plate_1_palm_lower_joint: type fixed, parent palm_lower, child plate_1_palm_lower, origin xyz=0 0 0 rpy=0 0 0
- added joint plate_1_thumb_fingertip_joint: type fixed, parent thumb_fingertip, child plate_1_thumb_fingertip, origin xyz=0 0 0 rpy=0 0 0
- added joint plate_20_palm_lower_joint: type fixed, parent palm_lower, child plate_20_palm_lower, origin xyz=0 0 0 rpy=0 0 0
- added joint plate_21_palm_lower_joint: type fixed, parent palm_lower, child plate_21_palm_lower, origin xyz=0 0 0 rpy=0 0 0
- added joint plate_22_palm_lower_joint: type fixed, parent palm_lower, child plate_22_palm_lower, origin xyz=0 0 0 rpy=0 0 0
- added joint plate_23_palm_lower_joint: type fixed, parent palm_lower, child plate_23_palm_lower, origin xyz=0 0 0 rpy=0 0 0
- added joint plate_24_palm_lower_joint: type fixed, parent palm_lower, child plate_24_palm_lower, origin xyz=0 0 0 rpy=0 0 0
- added joint plate_25_palm_lower_joint: type fixed, parent palm_lower, child plate_25_palm_lower, origin xyz=0 0 0 rpy=0 0 0
- added joint plate_2_palm_lower_joint: type fixed, parent palm_lower, child plate_2_palm_lower, origin xyz=0 0 0 rpy=0 0 0
- added joint plate_2_thumb_fingertip_joint: type fixed, parent thumb_fingertip, child plate_2_thumb_fingertip, origin xyz=0 0 0 rpy=0 0 0
- added joint plate_3_palm_lower_joint: type fixed, parent palm_lower, child plate_3_palm_lower, origin xyz=0 0 0 rpy=0 0 0
- added joint plate_3_thumb_fingertip_joint: type fixed, parent thumb_fingertip, child plate_3_thumb_fingertip, origin xyz=0 0 0 rpy=0 0 0
- added joint plate_4_palm_lower_joint: type fixed, parent palm_lower, child plate_4_palm_lower, origin xyz=0 0 0 rpy=0 0 0
- added joint plate_4_thumb_fingertip_joint: type fixed, parent thumb_fingertip, child plate_4_thumb_fingertip, origin xyz=0 0 0 rpy=0 0 0
- added joint plate_5_palm_lower_joint: type fixed, parent palm_lower, child plate_5_palm_lower, origin xyz=0 0 0 rpy=0 0 0
- added joint plate_5_thumb_fingertip_joint: type fixed, parent thumb_fingertip, child plate_5_thumb_fingertip, origin xyz=0 0 0 rpy=0 0 0
- added joint plate_6_palm_lower_joint: type fixed, parent palm_lower, child plate_6_palm_lower, origin xyz=0 0 0 rpy=0 0 0
- added joint plate_6_thumb_fingertip_joint: type fixed, parent thumb_fingertip, child plate_6_thumb_fingertip, origin xyz=0 0 0 rpy=0 0 0
- added joint plate_7_palm_lower_joint: type fixed, parent palm_lower, child plate_7_palm_lower, origin xyz=0 0 0 rpy=0 0 0
- added joint plate_7_thumb_fingertip_joint: type fixed, parent thumb_fingertip, child plate_7_thumb_fingertip, origin xyz=0 0 0 rpy=0 0 0
- added joint plate_8_palm_lower_joint: type fixed, parent palm_lower, child plate_8_palm_lower, origin xyz=0 0 0 rpy=0 0 0
- added joint plate_8_thumb_fingertip_joint: type fixed, parent thumb_fingertip, child plate_8_thumb_fingertip, origin xyz=0 0 0 rpy=0 0 0
- added joint plate_9_palm_lower_joint: type fixed, parent palm_lower, child plate_9_palm_lower, origin xyz=0 0 0 rpy=0 0 0
- added joint plate_9_thumb_fingertip_joint: type fixed, parent thumb_fingertip, child plate_9_thumb_fingertip, origin xyz=0 0 0 rpy=0 0 0

File: assets/leap_hand/robot.urdf.xacro (robot description, xacro)
@@ -539,3 +539,37 @@
 <xacro:plate parent_link="fingertip_2"  id="11" x="-0.00975" y="-0.04" z="0.025" roll="0" pitch="-0.8" yaw="0.0"/>
 <xacro:plate parent_link="fingertip_3"  id="11" x="-0.00975" y="-0.04" z="0.025" roll="0" pitch="-0.8" yaw="0.0"/>
+<xacro:plate parent_link="palm_lower"   id="1"      x="-0.04" y="${-0.0925+(0.016*0)}" z="-0.0352" roll="0" pitch="0" yaw="0.0"/>
+<xacro:plate parent_link="palm_lower"   id="2"      x="-0.04" y="${-0.0925+(0.016*1)}" z="-0.0352" roll="0" pitch="0" yaw="0.0"/>
+<xacro:plate parent_link="palm_lower"   id="3"      x="-0.04" y="${-0.0925+(0.016*2)}" z="-0.0352" roll="0" pitch="0" yaw="0.0"/>
+<xacro:plate parent_link="palm_lower"   id="4"      x="-0.04" y="${-0.0925+(0.016*3)}" z="-0.0352" roll="0" pitch="0" yaw="0.0"/>
+<xacro:plate parent_link="palm_lower"   id="5"      x="-0.04" y="${-0.0925+(0.016*4)}" z="-0.0352" roll="0" pitch="0" yaw="0.0"/>
+<xacro:plate parent_link="palm_lower"   id="6"      x="-0.04" y="${-0.0925+(0.016*5)}" z="-0.0352" roll="0" pitch="0" yaw="0.0"/>
+<xacro:plate parent_link="palm_lower"   id="7"      x="-0.04" y="${-0.0925+(0.016*6)}" z="-0.0352" roll="0" pitch="0" yaw="0.0"/>
+<xacro:plate parent_link="palm_lower"   id="8"      x="-0.04" y="${-0.0925+(0.016*7)}" z="-0.0352" roll="0" pitch="0" yaw="0.0"/>
+<xacro:plate parent_link="palm_lower"   id="9"      x="-0.05" y="${-0.0925+(0.016*0)}" z="-0.0352" roll="0" pitch="0" yaw="0.0"/>
+<xacro:plate parent_link="palm_lower"   id="10"     x="-0.05" y="${-0.0925+(0.016*1)}" z="-0.0352" roll="0" pitch="0" yaw="0.0"/>
+<xacro:plate parent_link="palm_lower"   id="11"     x="-0.05" y="${-0.0925+(0.016*2)}" z="-0.0352" roll="0" pitch="0" yaw="0.0"/>
+<xacro:plate parent_link="palm_lower"   id="12"     x="-0.05" y="${-0.0925+(0.016*3)}" z="-0.0352" roll="0" pitch="0" yaw="0.0"/>
+<xacro:plate parent_link="palm_lower"   id="13"     x="-0.05" y="${-0.0925+(0.016*4)}" z="-0.0352" roll="0" pitch="0" yaw="0.0"/>
+<xacro:plate parent_link="palm_lower"   id="14"     x="-0.05" y="${-0.0925+(0.016*5)}" z="-0.0352" roll="0" pitch="0" yaw="0.0"/>
+<xacro:plate parent_link="palm_lower"   id="15"     x="-0.05" y="${-0.0925+(0.016*6)}" z="-0.0352" roll="0" pitch="0" yaw="0.0"/>
+<xacro:plate parent_link="palm_lower"   id="16"     x="-0.05" y="${-0.0925+(0.016*7)}" z="-0.0352" roll="0" pitch="0" yaw="0.0"/>
+<xacro:plate parent_link="palm_lower"   id="17"     x="-0.06" y="${-0.0925+(0.016*1)}" z="-0.0352" roll="0" pitch="0" yaw="0.0"/>
+<xacro:plate parent_link="palm_lower"   id="18"     x="-0.06" y="${-0.0925+(0.016*2)}" z="-0.0352" roll="0" pitch="0" yaw="0.0"/>
+<xacro:plate parent_link="palm_lower"   id="19"     x="-0.06" y="${-0.0925+(0.016*3)}" z="-0.0352" roll="0" pitch="0" yaw="0.0"/>
+<xacro:plate parent_link="palm_lower"   id="20"     x="-0.07" y="${-0.0925+(0.016*1)}" z="-0.0352" roll="0" pitch="0" yaw="0.0"/>
+<xacro:plate parent_link="palm_lower"   id="21"     x="-0.07" y="${-0.0925+(0.016*2)}" z="-0.0352" roll="0" pitch="0" yaw="0.0"/>
+<xacro:plate parent_link="palm_lower"   id="22"     x="-0.07" y="${-0.0925+(0.016*3)}" z="-0.0352" roll="0" pitch="0" yaw="0.0"/>
+<xacro:plate parent_link="palm_lower"   id="23"     x="-0.08" y="${-0.0925+(0.016*1)}" z="-0.0352" roll="0" pitch="0" yaw="0.0"/>
+<xacro:plate parent_link="palm_lower"   id="24"     x="-0.08" y="${-0.0925+(0.016*2)}" z="-0.0352" roll="0" pitch="0" yaw="0.0"/>
+<xacro:plate parent_link="palm_lower"   id="25"     x="-0.08" y="${-0.0925+(0.016*3)}" z="-0.0352" roll="0" pitch="0" yaw="0.0"/>
+<xacro:plate parent_link="thumb_fingertip"  id="1" x="+0.0025" y="-0.035" z="-0.00225" roll="0.0" pitch="0.0" yaw="0.0"/>
+<xacro:plate parent_link="thumb_fingertip"  id="2" x="-0.0025" y="-0.035" z="-0.00225" roll="0.0" pitch="0.0" yaw="0.0"/>
+<xacro:plate parent_link="thumb_fingertip"  id="3" x="-0.0075" y="-0.035" z="-0.00225" roll="0.0" pitch="-0.2" yaw="0.0"/>
+<xacro:plate parent_link="thumb_fingertip"  id="4" x="+0.0025" y="-0.045" z="-0.00225" roll="0.0" pitch="0.0" yaw="0.0"/>
+<xacro:plate parent_link="thumb_fingertip"  id="5" x="-0.0025" y="-0.045" z="-0.00225" roll="0.0" pitch="0.0" yaw="0.0"/>
+<xacro:plate parent_link="thumb_fingertip"  id="6" x="-0.0075" y="-0.045" z="-0.00225" roll="0.0" pitch="-0.2" yaw="0.0"/>
+<xacro:plate parent_link="thumb_fingertip"  id="7" x="+0.0025" y="-0.055" z="-0.00225" roll="0.0" pitch="0.0" yaw="0.0"/>
+<xacro:plate parent_link="thumb_fingertip"  id="8" x="-0.0025" y="-0.055" z="-0.00225" roll="0.0" pitch="0.0" yaw="0.0"/>
+<xacro:plate parent_link="thumb_fingertip"  id="9" x="-0.0075" y="-0.055" z="-0.0025" roll="0.2" pitch="-0.2" yaw="0.0"/>
 </robot>
